Commit message: 3/20 sub 1

File: class/class06/move_urdf/install/urdf_r2d2/share/urdf_r2d2/urdf/r2d2.urdf.xacro (robot description, xacro)
@@ -16,5 +16,5 @@
   <xacro:property name="leg_size" value="0.20 0.10 0.8"/>
   <xacro:property name="leg_origin" value="0 0 -0.3"/>
-  <xacro:property name="leg_y" value="0.30"/>
+  <xacro:property name="leg_y" value="0.40"/>
   <xacro:property name="body_radius" value="0.20"/>
   <xacro:property name="body_length" value="0.6"/>
@@ -96,5 +96,5 @@
     <xacro:unit_inertial/>
     <visual>
-      <origin xyz="0 0 0" rpy="0 0 0"/>
+      <origin xyz="0 0 0.35" rpy="0 0 0"/>
       <geometry><sphere radius="${head_radius}"/></geometry>
       <material name="white"/>

File: class/class06/my_urdf/install/my_urdf/share/my_urdf/urdf/myfirst.urdf (robot description, URDF)
Before this commit: robot myfirst, 1 links, 0 joints
Links:
- link base_link: geometry collision box size=0.4 0.3 0.2; visual box size=0.4 0.3 0.2
